File: PCB/RECEPTEUR/kkap-recepteur.sch (KiCad schematic (older format))
At the start: 18 parts, among them IC1 ATMEGA328-P, P1 VIDEO, P2 ISP, P3 SERVO_PAN, P4 SERVO_TILT, P5 CHDK, P6 ALIM, P7 SP_SAT, U1 LM7805CT, U2 AP111733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

Commit message: PCB V1
Parts:
- removed C3: 0.1µF, symbol CP1
- removed P6: ALIM, symbol CONN_01X04
- added P6: BATT, Pin_Headers:Pin_Header_Straight_1x02_Pitch2.54mm, symbol CONN_01X02
- C1, C2, C4: footprint (none) -> Capacitors_ThroughHole:C_Radial_D5_L6_P2.5
- C5, C6: footprint (none) -> Capacitors_ThroughHole:C_Disc_D3_P2.5
- IC1: footprint DIL28 -> Housings_DIP:DIP-28_W7.62mm_Socket_LongPads
- P1, P3, P4, P7: footprint (none) -> Pin_Headers:Pin_Header_Straight_1x03_Pitch2.54mm
- P2: footprint (none) -> Pin_Headers:Pin_Header_Straight_2x03_Pitch2.54mm
- P5: footprint (none) -> Pin_Headers:Pin_Header_Straight_1x04_Pitch2.54mm
- R1: footprint (none) -> Resistors_ThroughHole:Resistor_Horizontal_RM7mm
- U1: footprint TO-220 -> Power_Integrations:TO-220
- Y1: footprint (none) -> Crystals:Crystal_HC49-U_Vertical
Connections:
- net +3V3: now also P7.2 (P2); no longer P7.1 (P1)
- net +5V: now also P5.2 (P2); no longer IC1.21 (AREF), P5.1 (P1)
- net +BATT: now also P1.2 (P2), P6.1 (P1); no longer P1.1 (P1)
- net CHDK_SIGNAL: now also P5.4 (P4); no longer P5.3 (P3)
- net GND: now also P1.1 (P1), P5.1 (P1), P7.1 (P1), P6.2 (P2); no longer P1.2 (P2), P5.2 (P2), P7.2 (P2)
- net SERVO_PAN: now also IC1.16 ((PCINT2/OC1B/~SS~)PB2); no longer IC1.14 ((PCINT0/CLKO/ICP1)PB0)
- net VIDEO_SIGNAL: now also P5.3 (P3); no longer P5.4 (P4)
