File: PCB/RECEPTEUR/kkap-recepteur.kicad_pcb (KiCad board)
At the start: 2 copper layers, 48.3 x 63.5 mm, 21 parts, among them IC1 ATMEGA328-P, P1 VIDEO, P2 ISP, P3 SERVO_PAN, P4 SERVO_TILT, P5 CHDK, P6 BATT, P7 SP_SAT, U1 LM7805CT, U2 AP111733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

Commit message: Modification du sat
Modification du pin header par un connecteur JST-ZH pour le satellite spektrum
Parts:
- P7: footprint Pin_Headers:Pin_Header_Straight_1x03_Pitch2.54mm -> JST_conn:JST-ZH-B3B-ZR
- moved P7 1.27 mm to (81.3, 45.7), turned to 270 degrees
Routing:
- net /SAT_TX: track 72.0 -> 75.6 mm
- net +5V: track 110.3 -> 111.2 mm
- net +3V3: track 43.8 -> 42.9 mm
Changed lines of the file:
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@@
     (area 40.304999 12.54 104.37 85.405)
     (thickness 1.6)
-    (drawings 12)
-    (tracks 106)
+    (drawings 8)
+    (tracks 107)
     (zones 0)
     (modules 21)
@@
     (model Pin_Headers.3dshapes/Pin_Header_Straight_1x04_Pitch2.54mm.wrl
       (at (xyz 0 -0.15 0))
-      (scale (xyz 1 1 1))
-      (rotate (xyz 0 0 90))
-    )
-  )
-  (module Pin_Headers:Pin_Header_Straight_1x03_Pitch2.54mm (layer F.Cu)
-    (at 81.28 44.45)
-    (descr "Through hole straight pin header, 1x03, 2.54mm pitch, single row")
-    (tags "Through hole pin header THT 1x03 2.54mm single row")
-    (fp_text reference P7 (at 0 -2.39) (layer F.SilkS)
-      (effects (font (size 1 1) (thickness 0.15)))
-    )
-    (fp_text value SP_SAT (at 0 7.47) (layer F.Fab)
-      (effects (font (size 1 1) (thickness 0.15)))
-    )
-    (fp_line (start -1.27 -1.27) (end -1.27 6.35) (layer F.Fab) (width 0.1))
-    (fp_line (start -1.27 6.35) (end 1.27 6.35) (layer F.Fab) (width 0.1))
-    (fp_line (start 1.27 6.35) (end 1.27 -1.27) (layer F.Fab) (width 0.1))
-    (fp_line (start 1.27 -1.27) (end -1.27 -1.27) (layer F.Fab) (width 0.1))
-    (fp_line (start -1.39 1.27) (end -1.39 6.47) (layer F.SilkS) (width 0.12))
-    (fp_line (start -1.39 6.47) (end 1.39 6.47) (layer F.SilkS) (width 0.12))
-    (fp_line (start 1.39 6.47) (end 1.39 1.27) (layer F.SilkS) (width 0.12))
-    (fp_line (start 1.39 1.27) (end -1.39 1.27) (layer F.SilkS) (width 0.12))
-    (fp_line (start -1.39 0) (end -1.39 -1.39) (layer F.SilkS) (width 0.12))
-    (fp_line (start -1.39 -1.39) (end 0 -1.39) (layer F.SilkS) (width 0.12))
-    (fp_line (start -1.6 -1.6) (end -1.6 6.6) (layer F.CrtYd) (width 0.05))
-    (fp_line (start -1.6 6.6) (end 1.6 6.6) (layer F.CrtYd) (width 0.05))
-    (fp_line (start 1.6 6.6) (end 1.6 -1.6) (layer F.CrtYd) (width 0.05))
-    (fp_line (start 1.6 -1.6) (end -1.6 -1.6) (layer F.CrtYd) (width 0.05))
-    (pad 1 thru_hole rect (at 0 0) (size 1.7 1.7) (drill 1) (layers *.Cu *.Mask)
-      (net 1 GND))
-    (pad 2 thru_hole oval (at 0 2.54) (size 1.7 1.7) (drill 1) (layers *.Cu *.Mask)
-      (net 4 +3V3))
-    (pad 3 thru_hole oval (at 0 5.08) (size 1.7 1.7) (drill 1) (layers *.Cu *.Mask)
-      (net 9 /SAT_TX))
-    (model Pin_Headers.3dshapes/Pin_Header_Straight_1x03_Pitch2.54mm.wrl
-      (at (xyz 0 -0.1 0))
       (scale (xyz 1 1 1))
       (rotate (xyz 0 0 90))
@@
     (pad 1 thru_hole circle (at 0 0) (size 4.064 4.064) (drill 3.048) (layers *.Cu *.Mask))
   )
-  (target plus (at 38.1 17.78) (size 5) (width 0.15) (layer Edge.Cuts))
-  (target plus (at 91.44 17.78) (size 5) (width 0.15) (layer Edge.Cuts))
-  (target plus (at 91.44 86.36) (size 5) (width 0.15) (layer Edge.Cuts))
-  (target plus (at 38.1 86.36) (size 5) (width 0.15) (layer Edge.Cuts))
+  (module JST_conn:JST-ZH-B3B-ZR (layer F.Cu)
+    (at 81.28 45.72 270)
+    (fp_text reference P7 (at 0 -3.3 270) (layer F.SilkS)
+      (effects (font (size 1 1) (thickness 0.15)))
+    )
+    (fp_text value SP_SAT (at 0 -4.9 270) (layer F.Fab)
+      (effects (font (size 1 1) (thickness 0.15)))
+    )
+    (fp_line (start -3 -2.2) (end -3 1.3) (layer F.SilkS) (width 0.15))
+    (fp_line (start 3 -2.2) (end 3 1.3) (layer F.SilkS) (width 0.15))
+    (fp_line (start -3 1.3) (end 3 1.3) (layer F.SilkS) (width 0.15))
+    (fp_line (start 3 -2.2) (end -3 -2.2) (layer F.SilkS) (width 0.15))
+    (pad 1 thru_hole oval (at -1.5 0 270) (size 1.2 1.524) (drill 0.762) (layers *.Cu *.Mask)
+      (net 1 GND))
+    (pad 2 thru_hole oval (at 0 0 270) (size 1.2 1.524) (drill 0.762) (layers *.Cu *.Mask)
+      (net 4 +3V3))
+    (pad 3 thru_hole oval (at 1.5 0 270) (size 1.2 1.524) (drill 0.762) (layers *.Cu *.Mask)
+      (net 9 /SAT_TX))
+  )
   (dimension 48.26 (width 0.3) (layer Cmts.User)
     (gr_text "48,260 mm" (at 64.77 13.89) (layer Cmts.User)
@@
   (segment (start 78.74 49.53) (end 76.2 46.99) (width 0.8) (layer B.Cu) (net 2))
   (segment (start 78.74 51.435) (end 78.74 49.53) (width 0.8) (layer B.Cu) (net 2))
-  (segment (start 83.185 55.88) (end 78.74 51.435) (width 0.8) (layer B.Cu) (net 2))
-  (segment (start 83.185 60.96) (end 83.185 55.88) (width 0.8) (layer B.Cu) (net 2))
-  (segment (start 81.915 62.23) (end 83.185 60.96) (width 0.8) (layer B.Cu) (net 2))
+  (segment (start 83.82 55.88) (end 78.74 51.435) (width 0.8) (layer B.Cu) (net 2))
+  (segment (start 83.82 60.96) (end 83.82 55.88) (width 0.8) (layer B.Cu) (net 2))
+  (segment (start 81.915 62.23) (end 83.82 60.96) (width 0.8) (layer B.Cu) (net 2))
   (segment (start 66.28 32.995) (end 60.985 32.995) (width 0.8) (layer B.Cu) (net 2) (status 20))
   (segment (start 60.985 32.995) (end 60.96 33.02) (width 0.8) (layer B.Cu) (net 2) (status 30))
@@
   (segment (start 48.26 45.72) (end 49.53 46.99) (width 0.8) (layer B.Cu) (net 3))
   (segment (start 48.26 33.02) (end 55.88 33.02) (width 0.8) (layer B.Cu) (net 3) (status 20))
+  (segment (start 81.28 45.72) (end 83.82 45.72) (width 0.8) (layer B.Cu) (net 4))
+  (segment (start 82.55 26.67) (end 84.455 28.575) (width 0.8) (layer B.Cu) (net 4))
+  (segment (start 82.55 26.67) (end 76.835 26.67) (width 0.8) (layer B.Cu) (net 4))
+  (segment (start 84.455 45.085) (end 84.455 28.575) (width 0.8) (layer B.Cu) (net 4))
+  (segment (start 83.82 45.72) (end 84.455 45.085) (width 0.8) (layer B.Cu) (net 4))
   (segment (start 68.58 32.995) (end 68.58 26.695) (width 0.8) (layer B.Cu) (net 4))
-  (segment (start 76.835 26.67) (end 82.55 26.67) (width 0.8) (layer B.Cu) (net 4))
-  (segment (start 83.185 46.99) (end 81.28 46.99) (width 0.8) (layer B.Cu) (net 4))
-  (segment (start 84.455 45.72) (end 83.185 46.99) (width 0.8) (layer B.Cu) (net 4))
-  (segment (start 84.455 28.575) (end 84.455 45.72) (width 0.8) (layer B.Cu) (net 4))
-  (segment (start 82.55 26.67) (end 84.455 28.575) (width 0.8) (layer B.Cu) (net 4))
   (segment (start 68.58 26.695) (end 76.81 26.695) (width 0.8) (layer B.Cu) (net 4))
   (segment (start 76.81 26.695) (end 76.835 26.67) (width 0.8) (layer B.Cu) (net 4))
@@
   (segment (start 81.28 57.15) (end 81.28 58.42) (width 0.8) (layer B.Cu) (net 8))
   (segment (start 76.2 52.07) (end 81.28 57.15) (width 0.8) (layer B.Cu) (net 8))
-  (segment (start 81.28 49.53) (end 82.55 49.53) (width 0.8) (layer B.Cu) (net 9))
-  (segment (start 50.8 68.58) (end 50.8 66.04) (width 0.8) (layer B.Cu) (net 9))
+  (segment (start 85.09 51.435) (end 85.09 48.895) (width 0.8) (layer B.Cu) (net 9))
+  (segment (start 85.09 74.295) (end 85.09 51.435) (width 0.8) (layer B.Cu) (net 9))
+  (segment (start 85.09 74.295) (end 80.01 78.74) (width 0.8) (layer B.Cu) (net 9))
+  (segment (start 80.01 78.74) (end 55.88 78.74) (width 0.8) (layer B.Cu) (net 9))
+  (segment (start 55.88 78.74) (end 52.07 74.93) (width 0.8) (layer B.Cu) (net 9))
+  (segment (start 52.07 74.93) (end 52.07 69.85) (width 0.8) (layer B.Cu) (net 9))
   (segment (start 52.07 69.85) (end 50.8 68.58) (width 0.8) (layer B.Cu) (net 9))
-  (segment (start 52.07 74.93) (end 52.07 69.85) (width 0.8) (layer B.Cu) (net 9))
-  (segment (start 55.88 78.74) (end 52.07 74.93) (width 0.8) (layer B.Cu) (net 9))
-  (segment (start 80.01 78.74) (end 55.88 78.74) (width 0.8) (layer B.Cu) (net 9))
-  (segment (start 84.455 74.295) (end 80.01 78.74) (width 0.8) (layer B.Cu) (net 9))
-  (segment (start 84.455 74.295) (end 84.455 51.435) (width 0.8) (layer B.Cu) (net 9))
-  (segment (start 82.55 49.53) (end 84.455 51.435) (width 0.8) (layer B.Cu) (net 9))
+  (segment (start 50.8 66.04) (end 50.8 68.58) (width 0.8) (layer B.Cu) (net 9))
+  (segment (start 83.415 47.22) (end 81.28 47.22) (width 0.8) (layer B.Cu) (net 9))
+  (segment (start 85.09 48.895) (end 83.415 47.22) (width 0.8) (layer B.Cu) (net 9))
   (segment (start 63.5 46.99) (end 61.595 46.99) (width 0.8) (layer B.Cu) (net 10))
   (segment (start 76.2 56.515) (end 76.2 58.42) (width 0.8) (layer B.Cu) (net 10))
@@
   (segment (start 73.66 58.42) (end 73.66 55.88) (width 0.8) (layer B.Cu) (net 11))
   (segment (start 66.04 52.07) (end 66.04 49.53) (width 0.8) (layer B.Cu) (net 11))
-  (segment (start 67.31 53.34) (end 66.04 52.07) (width 0.8) (layer B.Cu) (net 11))
-  (segment (start 71.12 53.34) (end 67.31 53.34) (width 0.8) (layer B.Cu) (net 11))
-  (segment (start 73.66 55.88) (end 71.12 53.34) (width 0.8) (layer B.Cu) (net 11))
+  (segment (start 66.04 52.07) (end 66.04 52.07) (width 0.8) (layer B.Cu) (net 11))
+  (segment (start 69.85 52.07) (end 66.04 52.07) (width 0.8) (layer B.Cu) (net 11))
+  (segment (start 73.66 55.88) (end 69.85 52.07) (width 0.8) (layer B.Cu) (net 11))
   (segment (start 66.04 46.99) (end 67.945 46.99) (width 0.8) (layer B.Cu) (net 12))
-  (segment (start 71.12 57.15) (end 71.12 58.42) (width 0.8) (layer B.Cu) (net 12))
-  (segment (start 69.85 55.88) (end 71.12 57.15) (width 0.8) (layer B.Cu) (net 12))
-  (via (at 69.85 55.88) (size 1.2) (drill 0.8) (layers F.Cu B.Cu) (net 12))
-  (segment (start 69.85 52.07) (end 69.85 55.88) (width 0.8) (layer F.Cu) (net 12))
-  (via (at 69.85 52.07) (size 1.2) (drill 0.8) (layers F.Cu B.Cu) (net 12))
-  (segment (start 68.58 50.8) (end 69.85 52.07) (width 0.8) (layer B.Cu) (net 12))
-  (segment (start 68.58 47.625) (end 68.58 50.8) (width 0.8) (layer B.Cu) (net 12))
+  (segment (start 71.12 55.88) (end 71.12 58.42) (width 0.8) (layer B.Cu) (net 12))
+  (segment (start 68.58 53.975) (end 71.12 55.88) (width 0.8) (layer B.Cu) (net 12))
+  (via (at 68.58 53.975) (size 1.2) (drill 0.8) (layers F.Cu B.Cu) (net 12))
+  (segment (start 68.58 49.53) (end 68.58 53.975) (width 0.8) (layer F.Cu) (net 12))
+  (via (at 68.58 49.53) (size 1.2) (drill 0.8) (layers F.Cu B.Cu) (net 12))
+  (segment (start 68.58 49.53) (end 68.58 49.53) (width 0.8) (layer B.Cu) (net 12))
+  (segment (start 68.58 47.625) (end 68.58 49.53) (width 0.8) (layer B.Cu) (net 12))
   (segment (start 67.945 46.99) (end 68.58 47.625) (width 0.8) (layer B.Cu) (net 12))
   (segment (start 55.88 52.07) (end 58.42 52.07) (width 0.8) (layer B.Cu) (net 13))
